Commit message: Make wheels continuous joints

File: src/papa_description/urdf/arlo.urdf.xacro (robot description, xacro)
@@ -2,4 +2,10 @@
 <robot name="arlobot" xmlns:xacro="http://ros.org/wiki/xacro">
   <!-- Macro for ArloBot body. -->
+  <!-- original radius 0.0762 original width 0.03175-->
+  <property name="wheel_radius" value="0.0775" />
+  <property name="wheel_width" value="0.0388" />
+  <property name="plate_height" value="0.1085" />
+  <property name="axis_height" value="${wheel_radius - plate_height}" />
+  <property name="wheel_base" value="0.160" />
   <property name="base_x" value="0.33" />
   <property name="base_y" value="0.33" />
@@ -24,10 +30,14 @@
       </visual>
     </link>
+    <joint name="base_footprint_joint" type="fixed">
+      <origin xyz="0 0 0.10125" rpy="0 0 0" />
+      <parent link="base_footprint"/>
+      <child link="base_link" />
+    </joint>
     <link name="base_link">
       <inertial>
         <mass value="2" />
         <origin xyz="0 0 0.0" />
-        <inertia ixx="0.01" ixy="0.0" ixz="0.0"
-          iyy="0.01" iyz="0.0" izz="0.5" />
+        <inertia ixx="0.01" ixy="0.0" ixz="0.0" iyy="0.01" iyz="0.0" izz="0.5" />
       </inertial>
       <visual>
@@ -45,5 +55,5 @@
       </collision>
     </link>
-    <link name="front_caster">
+    <link name="front_caster_link">
       <inertial>
         <mass value="0.001" />
@@ -66,7 +76,7 @@
       <origin xyz="0.18745 0 -0.00475" rpy="0 0 0" />
       <parent link="base_link" />
-      <child link="front_caster" />
+      <child link="front_caster_link" />
     </joint>
-    <link name="rear_caster">
+    <link name="rear_caster_link">
       <inertial>
         <mass value="0.001" />
@@ -89,64 +99,5 @@
       <origin xyz="-0.18745 0 -0.00475" rpy="0 0 0" />
       <parent link="base_link" />
-      <child link="rear_caster" />
-    </joint>
-    <joint name="base_footprint_joint" type="fixed">
-      <origin xyz="0 0 0.10125" rpy="0 0 0" />
-      <parent link="base_footprint"/>
-      <child link="base_link" />
-    </joint>
-    <link name="left_axle_link">
-      <inertial>
-        <origin xyz="0 0 0"/>
-        <mass value="0.01" />
-        <inertia ixx="0.001" ixy="0.0" ixz="0.0"
-          iyy="0.001" iyz="0.0" izz="0.001" />
-      </inertial>
-      <visual>
-        <origin xyz="0 0 0" rpy="0 1.5707 1.5707" />
-        <geometry>
-          <cylinder radius="0.00635" length = "0.00635"/>
-        </geometry>
-        <material name ="light_grey" />
-      </visual>
-      <collision>
-        <origin xyz="0 0 0" rpy="0 1.5707 1.5707" />
-        <geometry>
-          <cylinder radius="0.00635" length = "0.00635"/>
-        </geometry>
-      </collision>
-    </link>
-    <joint name="left_axle_joint" type="fixed">
-      <origin xyz="0 0.171475 0.0178" rpy="0 0 0"/>
-      <parent link="base_link"/>
-      <child link="left_axle_link"/>
-      <axis xyz="0 1 0"/>
-    </joint>
-    <link name="right_axle_link">
-      <inertial>
-        <origin xyz="0 0 0"/>
-        <mass value="0.01" />
-        <inertia ixx="0.001" ixy="0.0" ixz="0.0"
-          iyy="0.001" iyz="0.0" izz="0.001" />
-      </inertial>
-      <visual>
-        <origin xyz="0 0 0" rpy="0 1.5707 1.5707" />
-        <geometry>
-          <cylinder radius="0.00635" length = "0.00635"/>
-        </geometry>
-        <material name ="light_grey" />
-      </visual>
-      <collision>
-        <origin xyz="0 0 0" rpy="0 1.5707 1.5707" />
-        <geometry>
-          <cylinder radius="0.00635" length = "0.00635"/>
-        </geometry>
-      </collision>
-    </link>
-    <joint name="right_axle_joint" type="fixed">
-      <origin xyz="0 -0.171475 0.0178" rpy="0 0 0"/>
-      <parent link="base_link"/>
-      <child link="right_axle_link"/>
-      <axis xyz="0 1 0"/>
+      <child link="rear_caster_link" />
     </joint>
     <link name="left_wheel_link">
@@ -154,11 +105,10 @@
         <origin xyz="0 0 0"/>
         <mass value="0.01" />
-        <inertia ixx="0.001" ixy="0.0" ixz="0.0"
-          iyy="0.001" iyz="0.0" izz="0.001" />
+        <inertia ixx="0.001" ixy="0.0" ixz="0.0" iyy="0.001" iyz="0.0" izz="0.001" />
       </inertial>
       <visual>
         <origin xyz="0 0 0" rpy="0 1.5707 1.5707" />
         <geometry>
-          <cylinder radius="0.0762" length = "0.03175"/>
+          <cylinder radius="${wheel_radius}" length = "${wheel_width}"/>
         </geometry>
         <material name ="black" />
@@ -167,5 +117,5 @@
         <origin xyz="0 0 0" rpy="0 1.5707 1.5707" />
         <geometry>
-          <cylinder radius="0.0762" length = "0.03175"/>
+          <cylinder radius="${wheel_radius}" length = "${wheel_width}"/>
         </geometry>
       </collision>
@@ -173,9 +123,10 @@
     <!-- Fixed because we never rotate it anyway, it is just for show -->
     <!-- NOTE This may prevent gazebo from working with this model -->
-    <joint name="left_wheel_joint" type="fixed">
-      <origin xyz="0 0.01905 0" rpy="0 0 0"/>
-      <parent link="left_axle_link"/>
+    <joint name="left_wheel_joint" type="continuous">
+      <axis xyz="0 1 0"/>
+      <limit effort="10000.0" velocity="2"/>
+      <origin xyz="0 -${wheel_base} ${axis_height}" rpy="0 0 0"/>
+      <parent link="base_link"/>
       <child link="left_wheel_link"/>
-      <axis xyz="0 1 0"/>
     </joint>
     <link name="right_wheel_link">
@@ -200,51 +151,11 @@
       </collision>
     </link>
-    <!-- Fixed because we never rotate it anyway, it is just for show -->
-    <!-- NOTE This may prevent gazebo from working with this model -->
-    <joint name="right_wheel_joint" type="fixed">
-      <origin xyz="0 -0.01905 0" rpy="0 0 0"/>
-      <parent link="right_axle_link"/>
+    <joint name="right_wheel_joint" type="continuous">
+      <axis xyz="0 1 0"/>
+      <limit effort="10000.0" velocity="2"/>
+      <origin xyz="0 ${wheel_base} ${axis_height}" rpy="0 0 0"/>
+      <parent link="base_link"/>
       <child link="right_wheel_link"/>
-      <axis xyz="0 1 0"/>
     </joint>
-    <!-- This pretends to be in the center in order to aid in calculating degrees from multiple sensors on one fake laser scan -->
-    <joint name="ping_array_joint" type="fixed">
-      <origin xyz="0 0 0.03695" rpy="0 0 0" />
-      <parent link="base_link" />
-      <child link="ping_sensor_array" />
-    </joint>
-    <link name="ping_sensor_array">
-      <visual>
-        <geometry>
-          <box size="0.0174 0.06 0.0644" />
-        </geometry>
-      </visual>
-      <inertial>
-        <mass value="0.001" />
-        <origin xyz="0 0 0" />
-        <inertia ixx="0.0001" ixy="0.0" ixz="0.0"
-          iyy="0.0001" iyz="0.0"
-          izz="0.0001" />
-      </inertial>
-    </link>
-    <joint name="ir_array_joint" type="fixed">
-      <origin xyz="0 0 0.03695" rpy="0 0 0" />
-      <parent link="base_link" />
-      <child link="ir_sensor_array" />
-    </joint>
-    <link name="ir_sensor_array">
-      <visual>
-        <geometry>
-          <box size="0.0174 0.06 0.0644" />
-        </geometry>
-      </visual>
-      <inertial>
-        <mass value="0.001" />
-        <origin xyz="0 0 0" />
-        <inertia ixx="0.0001" ixy="0.0" ixz="0.0"
-          iyy="0.0001" iyz="0.0"
-          izz="0.0001" />
-      </inertial>
-    </link>
   </xacro:macro>
 </robot>

Commit message: Add navigation and kinect configuration

File: src/papa_description/urdf/arlo.urdf.xacro (robot description, xacro)
@@ -54,4 +54,11 @@
         </geometry>
       </collision>
+    </link>
+    <joint name="base_device_joint" type="fixed">
+      <origin xyz="0.10 0 0.10" rpy="0 0 0" />
+      <parent link="base_link"/>
+      <child link="device" />
+    </joint>
+    <link name="device">
     </link>
     <link name="front_caster_link">

File: src/papa_description/urdf/papa.urdf.xacro (robot description, xacro)
@@ -4,4 +4,33 @@
   <!-- There is no actual ArloBot model, I never made one. -->
   <xacro:include filename="$(find papa_description)/urdf/arlo.urdf.xacro"/>
+  <xacro:include filename="$(find turtlebot_description)/urdf/turtlebot_common_library.urdf.xacro" />
+  <xacro:include filename="$(find turtlebot_description)/urdf/stacks/hexagons.urdf.xacro"/>
+  <xacro:include filename="$(find turtlebot_description)/urdf/sensors/kinect.urdf.xacro"/>
+  <kobuki/>
+  <sensor_kinect  parent="base_link"/>
+  <joint name="right_sonar_base_link_joint" type="fixed">
+    <origin xyz="0.3 -0.08 0.10125" rpy="0 0 -0.610866667" />
+    <parent link="base_link"/>
+    <child link="right_sonar_link" />
+  </joint>
+  <link name="right_sonar_link">
+    <inertial>
+      <mass value="0.1" />
+      <origin xyz="0 0 0.0" />
+      <inertia ixx="0.01" ixy="0.0" ixz="0.0" iyy="0.01" iyz="0.0" izz="0.5" />
+    </inertial>
+  </link>
+  <joint name="left_sonar_base_link_joint" type="fixed">
+    <origin xyz="0.3 0.08 0.10125" rpy="0 0 0.610866667" />
+    <parent link="base_link"/>
+    <child link="left_sonar_link" />
+  </joint>
+  <link name="left_sonar_link">
+    <inertial>
+      <mass value="0.1" />
+      <origin xyz="0 0 0.0" />
+      <inertia ixx="0.01" ixy="0.0" ixz="0.0" iyy="0.01" iyz="0.0" izz="0.5" />
+    </inertial>
+  </link>
   <arlo_base/>
 </robot>

Commit message: Fix TF and odom publisher

File: src/papa_description/urdf/arlo.urdf.xacro (robot description, xacro)
@@ -29,4 +29,9 @@
         <material name="Green" />
       </visual>
+      <inertial>
+        <mass value="0.1" />
+        <origin xyz="0 0 0.0" />
+        <inertia ixx="0.01" ixy="0.0" ixz="0.0" iyy="0.01" iyz="0.0" izz="0.5" />
+      </inertial>
     </link>
     <joint name="base_footprint_joint" type="fixed">
@@ -54,11 +59,4 @@
         </geometry>
       </collision>
-    </link>
-    <joint name="base_device_joint" type="fixed">
-      <origin xyz="0.10 0 0.10" rpy="0 0 0" />
-      <parent link="base_link"/>
-      <child link="device" />
-    </joint>
-    <link name="device">
     </link>
     <link name="front_caster_link">

File: src/papa_description/urdf/papa.urdf.xacro (robot description, xacro)
@@ -5,8 +5,5 @@
   <xacro:include filename="$(find papa_description)/urdf/arlo.urdf.xacro"/>
   <xacro:include filename="$(find turtlebot_description)/urdf/turtlebot_common_library.urdf.xacro" />
-  <xacro:include filename="$(find turtlebot_description)/urdf/stacks/hexagons.urdf.xacro"/>
-  <xacro:include filename="$(find turtlebot_description)/urdf/sensors/kinect.urdf.xacro"/>
-  <kobuki/>
-  <sensor_kinect  parent="base_link"/>
+  <!-- Sonar links -->
   <joint name="right_sonar_base_link_joint" type="fixed">
     <origin xyz="0.3 -0.08 0.10125" rpy="0 0 -0.610866667" />
@@ -33,4 +30,53 @@
     </inertial>
   </link>
+  <!-- Kinect links -->
+  <joint name="camera_link_base_link_joint" type="fixed">
+    <origin xyz="0.0 0.0 0.10125" rpy="0 0 0" />
+    <parent link="base_link"/>
+    <child link="camera_link" />
+  </joint>
+  <link name="camera_link">
+    <visual>
+      <geometry>
+        <box size="0.064 0.121 0.0381" />
+      </geometry>
+      <material name="Blue" />
+    </visual>
+    <inertial>
+      <mass value="0.0001" />
+      <origin xyz="0 0 0" />
+      <inertia ixx="0.0001" ixy="0.0" ixz="0.0"
+               iyy="0.0001" iyz="0.0"
+               izz="0.0001" />
+    </inertial>
+  </link>
+  <joint name="camera_depth_joint" type="fixed">
+    <origin xyz="0 0.028 0" rpy="0 0 0" />
+    <parent link="camera_link" />
+    <child link="camera_depth_frame" />
+  </joint>
+  <link name="camera_depth_frame">
+    <inertial>
+        <mass value="0.0001" />
+        <origin xyz="0 0 0" />
+        <inertia ixx="0.0001" ixy="0.0" ixz="0.0"
+               iyy="0.0001" iyz="0.0"
+               izz="0.0001" />
+    </inertial>
+  </link>
+  <joint name="depth_optical_joint" type="fixed">
+    <origin xyz="0 0 0" rpy="${-M_PI/2} 0 ${-M_PI/2}" />
+    <parent link="camera_depth_frame" />
+    <child link="camera_depth_optical_frame" />
+  </joint>
+  <link name="camera_depth_optical_frame">
+    <inertial>
+        <mass value="0.0001" />
+        <origin xyz="0 0 0" />
+        <inertia ixx="0.0001" ixy="0.0" ixz="0.0"
+                 iyy="0.0001" iyz="0.0"
+                 izz="0.0001" />
+    </inertial>
+  </link>
   <arlo_base/>
 </robot>
